File: weather_station/weather_station.sch (KiCad schematic (older format))
At the start: 12 parts, among them J1 RJ11-6, J2 RJ11-6, J3 1935161, U1 BME280

Commit message: hardware update, add datasheets
Parts:
- removed B1: ESP32_THING_W_ANT_KEEPOUT, Boards:ESP32_THING, symbol SparkFun-Boards:ESP32_THING_W_ANT_KEEPOUT
- added U2: ESP32-DEVKITC-32D, weather_station:MODULE_ESP32-DEVKITC-32D, symbol ESP32-DEVKITC-32D:ESP32-DEVKITC-32D
Changed lines of the file:
@@
-$EndComp
-$Comp
-L SparkFun-Boards:ESP32_THING_W_ANT_KEEPOUT B1
-U 1 1 5F14CD04
-P 5000 4150
-F 0 "B1" H 5000 5510 45  0000 C CNN
-F 1 "ESP32_THING_W_ANT_KEEPOUT" H 5000 5426 45  0000 C CNN
-F 2 "Boards:ESP32_THING" H 5000 5350 20  0001 C CNN
-F 3 "" H 5000 4150 50  0001 C CNN
-F 4 "DEV-13907" H 5000 5331 60  0000 C CNN "Field4"
-	1    5000 4150
-	1    0    0    -1
 $EndComp
 $Comp
@@
 $EndComp
 $Comp
-L power:GND #PWR?
+L power:GND #PWR0106
 U 1 1 5F1C0B08
 P 1850 4600
-F 0 "#PWR?" H 1850 4350 50  0001 C CNN
+F 0 "#PWR0106" H 1850 4350 50  0001 C CNN
 F 1 "GND" H 1855 4427 50  0000 C CNN
 F 2 "" H 1850 4600 50  0001 C CNN
@@
 Connection ~ 1850 4000
 $Comp
-L power:VDD #PWR?
+L power:VDD #PWR0107
 U 1 1 5F1C797B
 P 8050 3650
-F 0 "#PWR?" H 8050 3500 50  0001 C CNN
+F 0 "#PWR0107" H 8050 3500 50  0001 C CNN
 F 1 "VDD" H 8065 3823 50  0000 C CNN
 F 2 "" H 8050 3650 50  0001 C CNN
@@
 $EndComp
 $Comp
-L power:GND #PWR?
+L power:GND #PWR0108
 U 1 1 5F1C7E8A
 P 8050 4350
-F 0 "#PWR?" H 8050 4100 50  0001 C CNN
+F 0 "#PWR0108" H 8050 4100 50  0001 C CNN
 F 1 "GND" H 8055 4177 50  0000 C CNN
 F 2 "" H 8050 4350 50  0001 C CNN
@@
 	8900 4200 8900 4400
 $Comp
-L power:VDD #PWR?
+L power:VDD #PWR0109
 U 1 1 5F1E26D9
 P 8550 3650
-F 0 "#PWR?" H 8550 3500 50  0001 C CNN
+F 0 "#PWR0109" H 8550 3500 50  0001 C CNN
 F 1 "VDD" H 8565 3823 50  0000 C CNN
 F 2 "" H 8550 3650 50  0001 C CNN
@@
 $EndComp
 $Comp
-L power:VDD #PWR?
+L power:VDD #PWR0110
 U 1 1 5F1E2DE8
 P 8900 3650
-F 0 "#PWR?" H 8900 3500 50  0001 C CNN
+F 0 "#PWR0110" H 8900 3500 50  0001 C CNN
 F 1 "VDD" H 8915 3823 50  0000 C CNN
 F 2 "" H 8900 3650 50  0001 C CNN
@@
 Text Label 8900 4400 0    50   ~ 0
 SCL
+$Comp
+L ESP32-DEVKITC-32D:ESP32-DEVKITC-32D U2
+U 1 1 5F49C879
+P 5000 4200
+F 0 "U2" H 5000 5367 50  0000 C CNN
+F 1 "ESP32-DEVKITC-32D" H 5000 5276 50  0000 C CNN
+F 2 "weather_station:MODULE_ESP32-DEVKITC-32D" H 5000 4200 50  0001 L BNN
+F 3 "Espressif Systems" H 5000 4200 50  0001 L BNN
+F 4 "4" H 5000 4200 50  0001 L BNN "Field4"
+	1    5000 4200
+	1    0    0    -1
+$EndComp
 $EndSCHEMATC

Commit message: add bme280 template
Parts:
- added C?: 10pF, Capacitor_SMD:C_0603_1608Metric_Pad1.05x0.95mm_HandSolder, symbol Device:C
- added R?: 100k, Resistor_SMD:R_0603_1608Metric_Pad1.05x0.95mm_HandSolder, symbol SparkFun-Resistors:RESISTOR0603
Connections:
- net labels added: RAIN
- wire segments 35 -> 60
Other:
- note added: "Anemometer & Wind Vane"
- note added: "Anemometer: Two inner conductors\nWind Vane: Two outer conductors"
- note added: "Rain Meter"
- note added: "Temperature & Humidity"
- moved on the sheet: C2, J3, R1, R2, U1
