File: weather_station/weather_station.sch (KiCad schematic (older format))
At the start: 14 parts, among them J1 RJ11-6, J2 RJ11-6, J3 1935161, U1 BME280, U2 ESP32-DEVKITC-32D

Commit message: schematic and pcb updates
Parts:
- added R4: 100k, Resistor_SMD:R_0603_1608Metric_Pad1.05x0.95mm_HandSolder, symbol SparkFun-Resistors:RESISTOR0603
- added R5: 4.7k, Resistor_SMD:R_0603_1608Metric_Pad1.05x0.95mm_HandSolder, symbol SparkFun-Resistors:RESISTOR0603
- gave numbers to parts that had none: 2
Connections:
- net labels added: WIND_DIR, WIND_SPD
- wire segments 60 -> 77
Changed lines of the file:
@@
 	2050 1900 2050 2250
 $Comp
-L Device:C C?
+L Device:C C1
 U 1 1 5F5253B2
 P 2050 2400
-F 0 "C?" H 2165 2446 50  0000 L CNN
+F 0 "C1" H 2165 2446 50  0000 L CNN
 F 1 "10pF" H 2165 2355 50  0000 L CNN
 F 2 "Capacitor_SMD:C_0603_1608Metric_Pad1.05x0.95mm_HandSolder" H 2088 2250 50  0001 C CNN
@@
 $EndComp
 $Comp
-L power:GND #PWR?
+L power:GND #PWR03
 U 1 1 5F5423A1
 P 2050 2800
-F 0 "#PWR?" H 2050 2550 50  0001 C CNN
+F 0 "#PWR03" H 2050 2550 50  0001 C CNN
 F 1 "GND" H 2055 2627 50  0000 C CNN
 F 2 "" H 2050 2800 50  0001 C CNN
@@
 	2050 2800 2050 2550
 $Comp
-L power:VDD #PWR?
+L power:VDD #PWR02
 U 1 1 5F50B5C4
 P 2050 1250
-F 0 "#PWR?" H 2050 1100 50  0001 C CNN
+F 0 "#PWR02" H 2050 1100 50  0001 C CNN
 F 1 "VDD" H 2065 1423 50  0000 C CNN
 F 2 "" H 2050 1250 50  0001 C CNN
@@
 $EndComp
 $Comp
-L SparkFun-Resistors:RESISTOR0603 R?
+L SparkFun-Resistors:RESISTOR0603 R3
 U 1 1 5F5102BE
 P 2050 1600
-F 0 "R?" H 2050 1800 45  0000 C CNN
+F 0 "R3" H 2050 1800 45  0000 C CNN
 F 1 "100k" H 2050 1700 45  0000 C CNN
 F 2 "Resistor_SMD:R_0603_1608Metric_Pad1.05x0.95mm_HandSolder" H 2050 1750 20  0001 C CNN
@@
 Text Label 2200 1900 0    50   ~ 0
 RAIN
-Wire Wire Line
-	4200 3700 4050 3700
-Text Label 4050 3700 0    50   ~ 0
+Text Label 3900 3700 0    50   ~ 0
 RAIN
 Wire Wire Line
@@
 Connection ~ 1700 2100
 $Comp
-L power:GND #PWR?
+L power:GND #PWR01
 U 1 1 5F562D2C
 P 1700 2350
-F 0 "#PWR?" H 1700 2100 50  0001 C CNN
+F 0 "#PWR01" H 1700 2100 50  0001 C CNN
 F 1 "GND" H 1705 2177 50  0000 C CNN
 F 2 "" H 1700 2350 50  0001 C CNN
@@
 Text Notes 3100 7750 0    50   ~ 0
 Temperature & Humidity
+$Comp
+L SparkFun-Resistors:RESISTOR0603 R5
+U 1 1 5F5CD842
+P 4300 1400
+F 0 "R5" H 4300 1600 45  0000 C CNN
+F 1 "4.7k" H 4300 1500 45  0000 C CNN
+F 2 "Resistor_SMD:R_0603_1608Metric_Pad1.05x0.95mm_HandSolder" H 4300 1550 20  0001 C CNN
+F 3 "" H 4300 1400 60  0001 C CNN
+F 4 " " H 4300 1521 60  0000 C CNN "Field4"
+	1    4300 1400
+	0    1    1    0
+$EndComp
+Wire Wire Line
+	3500 1650 4300 1650
+Wire Wire Line
+	4300 1650 4300 1600
+$Comp
+L power:VDD #PWR05
+U 1 1 5F5CF587
+P 4300 1100
+F 0 "#PWR05" H 4300 950 50  0001 C CNN
+F 1 "VDD" H 4315 1273 50  0000 C CNN
+F 2 "" H 4300 1100 50  0001 C CNN
+F 3 "" H 4300 1100 50  0001 C CNN
+	1    4300 1100
+	1    0    0    -1
+$EndComp
+Wire Wire Line
+	4300 1200 4300 1100
+Wire Wire Line
+	4300 1650 4500 1650
+Connection ~ 4300 1650
+Text Label 4500 1650 0    50   ~ 0
+WIND_DIR
+$Comp
+L power:GND #PWR06
+U 1 1 5F5D2AF1
+P 4300 2150
+F 0 "#PWR06" H 4300 1900 50  0001 C CNN
+F 1 "GND" H 4305 1977 50  0000 C CNN
+F 2 "" H 4300 2150 50  0001 C CNN
+F 3 "" H 4300 2150 50  0001 C CNN
+	1    4300 2150
+	1    0    0    -1
+$EndComp
+Wire Wire Line
+	3500 1950 3700 1950
+Wire Wire Line
+	4300 1950 4300 2150
+Wire Wire Line
+	3500 2050 3700 2050
+Wire Wire Line
+	3700 2050 3700 1950
+Connection ~ 3700 1950
+Wire Wire Line
+	3700 1950 4300 1950
+Wire Wire Line
+	3500 1750 3900 1750
+Text Label 4500 1750 0    50   ~ 0
+WIND_SPD
+Wire Wire Line
+	3500 1850 3700 1850
+Wire Wire Line
+	3700 1850 3700 1950
+Text Label 3900 3900 0    50   ~ 0
+WIND_SPD
+Text Label 3900 3800 0    50   ~ 0
+WIND_DIR
+Wire Wire Line
+	3900 3700 4200 3700
+Wire Wire Line
+	3900 3800 4200 3800
+Wire Wire Line
+	3900 3900 4200 3900
+$Comp
+L SparkFun-Resistors:RESISTOR0603 R4
+U 1 1 5F5E8AAF
+P 3900 1300
+F 0 "R4" H 3900 1500 45  0000 C CNN
+F 1 "100k" H 3900 1400 45  0000 C CNN
+F 2 "Resistor_SMD:R_0603_1608Metric_Pad1.05x0.95mm_HandSolder" H 3900 1450 20  0001 C CNN
+F 3 "" H 3900 1300 60  0001 C CNN
+F 4 " " H 3900 1421 60  0000 C CNN "Field4"
+	1    3900 1300
+	0    1    1    0
+$EndComp
+$Comp
+L power:VDD #PWR04
+U 1 1 5F5E960F
+P 3900 950
+F 0 "#PWR04" H 3900 800 50  0001 C CNN
+F 1 "VDD" H 3915 1123 50  0000 C CNN
+F 2 "" H 3900 950 50  0001 C CNN
+F 3 "" H 3900 950 50  0001 C CNN
+	1    3900 950
+	1    0    0    -1
+$EndComp
+Wire Wire Line
+	3900 950  3900 1100
+Wire Wire Line
+	3900 1500 3900 1750
+Connection ~ 3900 1750
+Wire Wire Line
+	3900 1750 4500 1750
 $EndSCHEMATC

Commit message: more pcb update
Parts:
- added C?: 10pF, Capacitor_SMD:C_0603_1608Metric_Pad1.05x0.95mm_HandSolder, symbol Device:C
Connections:
- wire segments 77 -> 80
Other:
- moved on the sheet: C2, R1, R2, U1

Commit message: add schematic pdf
Parts:
- gave numbers to parts that had none: 1
Changed lines of the file:
@@
 Wire Wire Line
 	1550 1800 1650 1800
-Text Notes 3200 2650 0    50   ~ 0
+Text Notes 3200 2700 0    50   ~ 0
 Anemometer: Two inner conductors\nWind Vane: Two outer conductors
 Wire Wire Line
@@
 	3900 1950 3900 2000
 $Comp
-L Device:C C?
+L Device:C C3
 U 1 1 5F63B6B2
 P 4300 2050
-F 0 "C?" H 4415 2096 50  0000 L CNN
+F 0 "C3" H 4415 2096 50  0000 L CNN
 F 1 "10pF" H 4415 2005 50  0000 L CNN
 F 2 "Capacitor_SMD:C_0603_1608Metric_Pad1.05x0.95mm_HandSolder" H 4338 1900 50  0001 C CNN
@@
 $EndComp
 $Comp
-L power:GND #PWR?
+L power:GND #PWR0113
 U 1 1 5F63BB57
 P 4300 2300
-F 0 "#PWR?" H 4300 2050 50  0001 C CNN
+F 0 "#PWR0113" H 4300 2050 50  0001 C CNN
 F 1 "GND" H 4305 2127 50  0000 C CNN
 F 2 "" H 4300 2300 50  0001 C CNN

Commit message: pcb updates and some tiny code changes
Parts:
- removed J1, J2: RJ11-6, Connectors:RJ11-6, symbol SparkFun-Connectors:RJ11-6
- added C4: 100nF, Capacitor_SMD:C_0603_1608Metric_Pad1.08x0.95mm_HandSolder, symbol Device:C
- added J1: 1935161, TerminalBlock_Phoenix:TerminalBlock_Phoenix_MKDS-1,5-2_1x02_P5.00mm_Horizontal, symbol dk_Terminal-Blocks-Wire-to-Board:1935161
- added J2: Screw_Terminal_01x03, TerminalBlock_Phoenix:TerminalBlock_Phoenix_MKDS-1,5-3_1x03_P5.00mm_Horizontal, symbol Connector:Screw_Terminal_01x03
- added R6: 1k, Resistor_SMD:R_0603_1608Metric_Pad0.98x0.95mm_HandSolder, symbol SparkFun-Resistors:RESISTOR0603
- added U3: S35770, Package_SO:SSOP-8_5.25x5.24mm_P1.27mm, symbol KevinsLib:S35770
- C1, C2, C3: footprint Capacitor_SMD:C_0603_1608Metric_Pad1.05x0.95mm_HandSolder -> Capacitor_SMD:C_0603_1608Metric_Pad1.08x0.95mm_HandSolder
- R1, R2, R3, R4, R5: footprint Resistor_SMD:R_0603_1608Metric_Pad1.05x0.95mm_HandSolder -> Resistor_SMD:R_0603_1608Metric_Pad0.98x0.95mm_HandSolder
Connections:
- wire segments 80 -> 84
- no-connect marks 0 -> 30
Other:
- note removed: "Anemometer: Two inner conductors\nWind Vane: Two outer conductors"
