File: weather_station/_autosave-weather_station.kicad_pcb (KiCad board)
At the start: 2 copper layers, 64.8 x 69.9 mm, 17 parts, among them J1 RJ11-6, J2 RJ11-6, J3 1935161, U1 BME280, U2 ESP32-DEVKITC-32D

Commit message: pcb updates, dont use this the schematic is scuffed
Routing:
- net /WIND_DIR: track 7.42 -> 35.9 mm
- net VDD: track 23.3 -> 43.0 mm, vias 2 -> 3
- net GND: track 11.3 -> 14.4 mm
Changed lines of the file:
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@@
     (thickness 1.6)
     (drawings 4)
-    (tracks 48)
+    (tracks 61)
     (zones 0)
     (modules 17)
@@
       (outputformat 1)
       (mirror false)
-      (drillshape 1)
+      (drillshape 0)
       (scaleselection 1)
-      (outputdirectory ""))
+      (outputdirectory "gerbers/"))
   )
   (net 0 "")
@@
   (segment (start 157.48 81.76) (end 157.48 83.82) (width 0.25) (layer F.Cu) (net 1))
   (via (at 157.48 83.82) (size 0.8) (drill 0.4) (layers F.Cu B.Cu) (net 1))
+  (segment (start 133.83 76.2) (end 133.35 75.72) (width 0.25) (layer F.Cu) (net 1))
+  (segment (start 138.43 76.2) (end 133.83 76.2) (width 0.25) (layer F.Cu) (net 1))
+  (segment (start 133.35 72.95) (end 127 66.6) (width 0.25) (layer F.Cu) (net 1))
+  (segment (start 133.35 75.72) (end 133.35 72.95) (width 0.25) (layer F.Cu) (net 1))
+  (via (at 156.21 67.31) (size 0.8) (drill 0.4) (layers F.Cu B.Cu) (net 1))
+  (segment (start 157.48 68.58) (end 156.21 67.31) (width 0.25) (layer F.Cu) (net 1))
+  (segment (start 157.48 69.37) (end 157.48 68.58) (width 0.25) (layer F.Cu) (net 1))
   (segment (start 163.83 78.2) (end 162.805 77.175) (width 0.25) (layer F.Cu) (net 2))
   (segment (start 163.83 81.28) (end 163.83 78.2) (width 0.25) (layer F.Cu) (net 2))
@@
   (segment (start 165.425 76.525) (end 166.37 77.47) (width 0.25) (layer F.Cu) (net 2))
   (segment (start 164.854999 76.525) (end 165.425 76.525) (width 0.25) (layer F.Cu) (net 2))
+  (segment (start 115.57 95.885) (end 116.84 95.885) (width 0.25) (layer F.Cu) (net 2))
+  (segment (start 114.3 97.155) (end 115.57 95.885) (width 0.25) (layer F.Cu) (net 2))
   (segment (start 156.92 71.68) (end 157.48 71.12) (width 0.25) (layer F.Cu) (net 4))
   (segment (start 152.4 71.68) (end 156.92 71.68) (width 0.25) (layer F.Cu) (net 4))
@@
   (segment (start 133.35 77.995) (end 132.045 79.3) (width 0.25) (layer F.Cu) (net 38))
   (segment (start 133.35 77.47) (end 133.35 77.995) (width 0.25) (layer F.Cu) (net 38))
+  (segment (start 116.84 100.965) (end 121.285 100.965) (width 0.25) (layer B.Cu) (net 38))
+  (segment (start 121.285 100.965) (end 123.19 99.06) (width 0.25) (layer B.Cu) (net 38))
+  (segment (start 123.19 83.11) (end 127 79.3) (width 0.25) (layer B.Cu) (net 38))
+  (segment (start 123.19 99.06) (end 123.19 83.11) (width 0.25) (layer B.Cu) (net 38))
   (segment (start 114.3 99.695) (end 112.395 99.695) (width 0.25) (layer F.Cu) (net 39))
   (segment (start 112.395 99.695) (end 111.76 99.06) (width 0.25) (layer F.Cu) (net 39))
